Commit message: working in my_big_bazu

File: big_bazu/urdf/my_big_bazu.urdf (robot description, URDF)
Before this commit: robot my_big_bazu, 8 links, 7 joints
Links:
- added link arm_2_link, mass 0.0; collision box size=0.035 0.08 0.017; visual box size=0.035 0.08 0.017
- added link arm_3_link, mass 0.0; collision box size=0.035 0.032 0.017; visual box size=0.035 0.032 0.017
- added link arm_4_base_link, mass 0.0; collision box size=0.035 0.05 0.017; visual box size=0.03 0.04 0.01
- added link arm_4_link, mass 0.0; collision box size=0.035 0.03 0.017; visual box size=0.03 0.03 0.01
- added link greifer_links, mass 0.0; collision box size=0.05 0.01 0.01; visual box size=0.05 0.01 0.01
- added link greifer_rechts, mass 0.0; collision box size=0.05 0.01 0.01; visual box size=0.05 0.01 0.01
- added link plate_3_link, mass 0.0; collision cylinder length=0.023 radius=0.0175; visual cylinder length=0.023 radius=0.0175
- added link plate_4_link, mass 0.0; collision cylinder length=0.023 radius=0.0175; visual cylinder length=0.023 radius=0.0175
- added link plate_5_link, mass 0.0; collision cylinder length=0.023 radius=0.0175; visual cylinder length=0.023 radius=0.0175
- added link plate_6_link, mass 0.0; collision cylinder length=0.013 radius=0.0175; visual cylinder length=0.013 radius=0.0175
- link arm_1_link: geometry collision box size=0.035 0.13 0.017; visual box size=0.035 0.13 0.017
- link plate_2_link: geometry collision cylinder length=0.023 radius=0.0175; visual cylinder length=0.023 radius=0.0175
Joints:
- removed joint joint_name
- removed joint teller_joint
- added joint arm_4_to_plate_joint: type fixed, parent plate_6_link, child arm_4_link, origin xyz=0.0 0.009 0.002 rpy=0.0 0.0 0.0
- added joint arm_base_joint: type fixed, parent arm_4_link, child arm_4_base_link, origin xyz=0.0 0.03 0.005 rpy=1.57 0.0 1.57
- added joint arm_lift_joint_2: type revolute, parent plate_1_link, child plate_2_link, origin xyz=0 0 0.013 rpy=0 0 1.17, axis 0 0 1, limit lower=-2.8 upper=0.35 effort=1000.0 velocity=50.0
- added joint arm_ratation_joint_4: type revolute, parent arm_2_link, child arm_3_link, origin xyz=0.0 0.056 0.0 rpy=0 0 0, axis 0 1 0, limit lower=0.0 upper=1.57 effort=1000.0 velocity=50.0
- added joint arm_to_arm_joint_3: type revolute, parent plate_3_link, child plate_4_link, origin xyz=0 0 -0.023 rpy=0 0 -2.6, axis 0 0 -1, limit lower=-2.35 upper=0.1 effort=1000.0 velocity=50.0
- added joint arm_to_nick_arm_joint_5: type revolute, parent plate_5_link, child plate_6_link, origin xyz=0 0 0.018 rpy=0 0 -0.14, axis 0 0 1, limit lower=-0.78 upper=0.78 effort=1000.0 velocity=50.0
- added joint arm_to_plate_2_joint: type fixed, parent arm_1_link, child plate_3_link, origin xyz=0.0 0.065 -0.003 rpy=0 0 0
- added joint arm_to_plate_4_joint: type fixed, parent plate_4_link, child arm_2_link, origin xyz=0.0 0.04 -0.003 rpy=0.0 0.0 0.0
- added joint greifer_joint_6: type prismatic, parent arm_4_base_link, child greifer_rechts, origin xyz=0.04 0.015 0 rpy=0 0 0, axis 0 1 0, limit lower=-0.006 upper=0.0 effort=1000.0 velocity=0.5
- added joint greifer_joint_7: type prismatic, parent arm_4_base_link, child greifer_links, origin xyz=0.04 -0.015 0 rpy=0 0 0, axis 0 1 0, limit lower=0.0 upper=0.008 effort=1000.0 velocity=0.5
- added joint plate_to_arm_3_joint: type fixed, parent arm_3_link, child plate_5_link, origin xyz=0.0 0.015 0.003 rpy=0 0 0
- added joint teller_joint_1: type revolute, parent body_link, child teller_link, origin xyz=0.0 0.0 0.029 rpy=0.0 0.0 0.0, axis 0.0 0.0 1.0, limit lower=-1.57 upper=1.57 effort=1000.0 velocity=50.0
- joint arm_to_plate_1_joint: origin xyz=0.0 0.065 0.0115 rpy=0.0 0.0 0.0 -> xyz=0.0 0.065 0.003 rpy=0.0 0.0 0.0

Commit message: working on gz

File: big_bazu/urdf/my_big_bazu.urdf (robot description, URDF)
Before this commit: robot my_big_bazu, 18 links, 17 joints
Links:
- link arm_1_link: mass 0.0 -> 0.3
- link arm_2_link: mass 0.0 -> 0.3
- link arm_3_link: mass 0.0 -> 0.1
- link arm_4_base_link: mass 0.0 -> 0.01
- link arm_4_link: mass 0.0 -> 0.02
- link base_link: mass 0.0 -> 10.0
- link body_link: mass 0.0 -> 1.0
- link greifer_links: mass 0.0 -> 0.01
- link greifer_rechts: mass 0.0 -> 0.01
- link plate_1_link: mass 0.0 -> 0.03
- link plate_2_link: mass 0.0 -> 0.03
- link plate_3_link: mass 0.0 -> 0.03
- link plate_4_link: mass 0.0 -> 0.03
- link plate_5_link: mass 0.0 -> 0.2
- link plate_6_link: mass 0.0 -> 0.02
- link ta_link: mass 0.0 -> 0.3
- link teller_link: mass 0.0 -> 0.3

Commit message: workflow

File: big_bazu/urdf/my_big_bazu.urdf (robot description, URDF)
Before this commit: robot my_big_bazu, 18 links, 17 joints
Links:
- link arm_1_link: mass 0.3 -> 0.0
- link arm_2_link: mass 0.3 -> 0.0
- link arm_3_link: mass 0.1 -> 0.0
- link arm_4_base_link: mass 0.01 -> 0.0
- link arm_4_link: mass 0.02 -> 0.0
- link base_link: mass 10.0 -> 0.0
- link body_link: mass 1.0 -> 0.0
- link greifer_links: mass 0.01 -> 0.0
- link greifer_rechts: mass 0.01 -> 0.0
- link plate_1_link: mass 0.03 -> 0.0
- link plate_2_link: mass 0.03 -> 0.0
- link plate_3_link: mass 0.03 -> 0.0
- link plate_4_link: mass 0.03 -> 0.0
- link plate_5_link: mass 0.2 -> 0.0
- link plate_6_link: mass 0.02 -> 0.0
- link ta_link: mass 0.3 -> 0.0
- link teller_link: mass 0.3 -> 0.0
Joints:
- joint arm_to_nick_arm_joint_5: limit lower=-0.78 upper=0.78 effort=1000.0 velocity=50.0 -> lower=-1.57 upper=1.57 effort=1000.0 velocity=50.0

Commit message: workflow

File: big_bazu/urdf/my_big_bazu.urdf (robot description, URDF)
Before this commit: robot my_big_bazu, 18 links, 17 joints
Links:
- link arm_1_link: mass 0.0 -> 0.02
- link arm_2_link: mass 0.0 -> 0.3
- link arm_3_link: mass 0.0 -> 0.3
- link arm_4_base_link: mass 0.0 -> 0.3
- link arm_4_link: mass 0.0 -> 0.3
- link base_link: mass 0.0 -> 1.0
- link body_link: mass 0.0 -> 3.0
- link greifer_links: mass 0.0 -> 0.02
- link greifer_rechts: mass 0.0 -> 0.03
- link plate_1_link: mass 0.0 -> 0.01
- link plate_2_link: mass 0.0 -> 0.3
- link plate_3_link: mass 0.0 -> 0.01
- link plate_4_link: mass 0.0 -> 0.01
- link plate_5_link: mass 0.0 -> 0.01
- link plate_6_link: mass 0.0 -> 0.01
- link ta_link: mass 0.0 -> 0.8
- link teller_link: mass 0.0 -> 0.5
